File: Termometria.kicad_sch (KiCad schematic)
At the start: 60 parts, among them J1 Current_sense, U10 74HC74, U11 NE555D, U16 MPY634KU, U17 CD4052B, U18 ADA4898-2, U19 CD4052B, U7 ADA4898-2, U8 ADA4898-2, U9 ADA4898-2

Commit message: first commit
Other:
- moved on the sheet: C31, C32, C33, C34, C35, C36, C37, C38, C39, C40, C41, C42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

Commit message: module created
Parts:
- removed C22, C23, C24, C25, C30, C42: C, symbol Device:C
- removed R17, R18, R19, R20, R21, R22, R23, R24: R, symbol Device:R
- removed R33, R35, R39, R40, R41, R42: 1k, symbol Device:R
- removed R34, R36: 2.2k, symbol Device:R
- removed U10: 74HC74, symbol 74xx:74HC74
- removed U11: NE555D, Package_SO:SOIC-8_3.9x4.9mm_P1.27mm, symbol Timer:NE555D
- removed U16: MPY634KU, Package_SO:SOIC-16W_7.5x10.3mm_P1.27mm, symbol Analog:MPY634KU
- removed U17, U19: CD4052B, symbol Analog_Switch:CD4052B
- removed unit 2 of U18
- removed unit 2 of U7
- removed unit 1 of U7
- removed unit 2 of U9
- removed unit 1 of U9
Connections:
- net A_AMP_OUT: now also U8.7
- net Amplifier Block/IN +: now also R10.2; no longer R10.1
- net Amplifier Block/IN -: now also R10.1; no longer R10.2
- no-connect marks 5 -> 0
Other:
- removed sheet Amplifier Block1
- note removed: "20Hz 50% duty waveform shaping"
- note removed: "40Hz Pulse Generator"
- note removed: "AD835"
- moved on the sheet: R10

Commit message: layout made
Parts:
- removed C32, C33, C34, C36, C37, C38, C39, C40, C41, C5: C, symbol Device:C
- removed R3, R5: R, symbol Device:R
- removed U18, U7, U8, U9: ADA4898-2, Package_SO:SOIC-8-1EP_3.9x4.9mm_P1.27mm_EP2.41x3.81mm, symbol Amplifier_Operational:ADA4898-2
- added J2: Power, Connector_PinHeader_2.54mm:PinHeader_1x03_P2.54mm_Vertical, symbol Connector:Conn_01x03_Pin
- added U4: NE5532, Package_SO:SOIC-8_3.9x4.9mm_P1.27mm, symbol Amplifier_Operational:NE5532
- C26, C27, C28, C29, C31, C35: footprint (none) -> Capacitor_SMD:C_0603_1608Metric
- J1: value Current_sense -> Conn_Coaxial; footprint (none) -> Connector_Coaxial:SMA_Amphenol_901-144_Vertical
- R10: footprint (none) -> Resistor_THT:R_Axial_DIN0414_L11.9mm_D4.5mm_P15.24mm_Horizontal
- R25, R26, R27, R28, R29, R30, R31, R32: footprint (none) -> Resistor_SMD:R_0603_1608Metric
- R4: value R -> 100k; footprint (none) -> Resistor_SMD:R_0603_1608Metric
Connections:
- net +15V: now also J2.1 (Pin_1), U4.8 (V+)
- net -15V: now also J2.3 (Pin_3), U4.4 (V-)
- net GND: now also J2.2 (Pin_2)
- net at C29.1, R31.1: now also U4.3 (+)
- net at C27.1, R27.2: now also U4.5 (+)
- net at R30.1, R32.2: now also U4.2 (-)
- net at C26.2, R28.1: now also J1.1 (In), U4.7
- net at R26.1, R28.2: now also U4.6 (-)
- net at R25.1: now also R29.2, R32.1, U4.1
