File: amplifier.kicad_sch (KiCad schematic)
At the start: 19 parts, among them U1 AD745, U2 AD745, U3 INA103

Commit message: first commit
Other:
- title: (none) -> Amplifier block
Changed lines of the file:
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@@
 (kicad_sch (version 20230121) (generator eeschema)
   (paper "A4")
+  (title_block
+    (title "Amplifier block")
+  )
   (junction (at 143.51 160.02) (diameter 0) (color 0 0 0 0)
   )

Commit message: layout made
Parts:
- removed C2: C, symbol Device:C
- removed C5, C6: 1u 25V, symbol Device:C_Polarized
- removed R2, R3: R, symbol Device:R
- added C1: 10n, Capacitor_SMD:C_0603_1608Metric, symbol Device:C
- added R1: 510, Resistor_SMD:R_0603_1608Metric, symbol Device:R
- added R1: 5.1k, Resistor_SMD:R_0603_1608Metric, symbol Device:R
- C1: value C -> 10n; footprint (none) -> Capacitor_SMD:C_0603_1608Metric
- C10, C11, C4, C7, C8, C9: footprint (none) -> Capacitor_SMD:C_0603_1608Metric
- R1: value R -> 5.1k; footprint (none) -> Resistor_SMD:R_0603_1608Metric
- R3: value 100 -> 50; footprint (none) -> Resistor_SMD:R_0603_1608Metric
- R6, R7: footprint (none) -> Resistor_SMD:R_0603_1608Metric
- U3: footprint Package_SO:SOIC-16W_7.5x10.3mm_P1.27mm -> Package_DIP:DIP-16_W7.62mm_LongPads
Connections:
- net at C1.1, R1.1, U1.12: now also U3.1 (+); no longer U3.16 (-)
- net at C1.2, R1.2, U1.3 (-): now also R1.1
- net at U2.12: now also U3.16 (-), C1.2, R1.2; no longer U3.1 (+)
- net at U2.3 (-): now also C1.1, R1.1, R1.2
